File: hw/projects/IMU_NoPilot/IMU_NoPilot.sch (EAGLE design)
At the start: 10 parts

Commit message: Finished Power and Reset part of schematics
Parts:
- added C10, C11: (no value), resistor:C-EUC0805
- added C12: 100n, resistor:C-EUC0805
- added R1, R2: 10k, resistor:R-EU_R0805
- added U$4: XTAL_5X3P2, misc_devices:XTAL_5X3P2
- added U$6, U$7: OMRON_B3FS_1000, misc_devices:OMRON_B3FS_1000
Connections:
- new net N$4: C10.1, U$1G$5.PORTH_0, U$4.Q1
- new net N$6: C11.1, U$1G$5.PORTH_1, U$4.Q2
- new net N$7: C12.1, R1.1, U$1G$1.!RST, U$6.P$2
- new net N$8: R2.2, U$1G$1.BOOT0, U$7.P$2
- net GND: now also C10.2, C11.2, C12.2, R2.1, U$1G$3.PORTB_2, U$4.GND, U$6.P$1
- net VDD: now also R1.2, U$7.P$1
Other:
- note added: "100n cap should be close to VDDA pin."
- note added: "100n caps should be close to VDD pins."
- note added: "BOOT1"

Commit message: added accelerometer, gyro and magnetometer to schematics. Not yet connected to the uC
Parts:
- added C13: 4.7u, resistor:C-EUC0805
- added C14: 0.22u, resistor:C-EUC0805
- added C15, C19: 10u, resistor:C-EUC0805
- added C16, C17, C18: 100n, resistor:C-EUC0805
- added C20: 10n (25V), resistor:C-EUC0805
- added U$12: LSM303DLHC, sensors:LSM303DLHC
- added U$13: LSM330DLC, sensors:LSM330DLC
Connections:
- new net DEN_GYRO: U$13.DEN_G
- new net DRDY_GYRO: U$13.DRDY_G
- new net I2C-1_SCL: U$12.SCL
- new net I2C-1_SDA: U$12.SDA
- new net INT1_ACCL: U$13.INT1_A
- new net INT1_GYRO: U$13.INT1_G
- new net INT2_ACCL: U$13.INT2_A
- new net LSM303-INT2: U$12.INT2
- new net LSM303_DRDY: U$12.DRDY
- new net LSM303_INT1: U$12.INT1
- new net N$10: C20.1, U$13.CAP
- new net N$3: C14.1, U$12.SETP
- new net N$5: C14.2, U$12.SETC
- new net N$9: C13.1, U$12.C1
- new net SPI_CLK: U$13.SCL
- new net SPI_CS_ACCL: U$13.!CS_A
- new net SPI_CS_GYRO: U$13.!CS_G
- new net SPI_MISO: U$13.SDO_A, U$13.SDO_G
- new net SPI_MOSI: U$13.SDA
- net GND: now also C13.2, C15.2, C16.2, C17.2, C18.2, C19.2, C20.2, U$12.GND, U$13.VSS
- net VDD: now also C15.1, C16.1, C17.1, C18.1, C19.1, U$12.VDD, U$12.VDD_IO, U$13.VDD, U$13.VDD_IO

Commit message: Ready for first try at autoroute. Nothing is properly reviewed yet
Parts:
- added C21: 4u7, resistor:C-EUC0805
- added C22: 10u, resistor:C-EUC0805
- added L1: MLB-160808-0060PQ, resistor:R-EU_R0603
- added P1: USB_MICRO_AB, connectors:USB_MICRO_AB
- added P2: ST_LINK, connectors:ST_LINK
- added P3: PWR3, connectors:PWR3
- added R3, R4: 330R, resistor:R-EU_R0805
- added R5, R6: 100, resistor:R-EU_R0805
- added R7, R8: 4k7, resistor:R-EU_R0805
- added U4: MPL3115A2, sensors:MPL3115A2
- added U5: MTK-3329, sensors:MTK-3329
- added U6: MCP1825, misc_devices:MCP1825
- C10: value (none) -> 4.7u
- C11: value (none) -> 100n
- C12: value 100n -> 0.22u
- C13: value 4.7u -> 10n (25V)
- C14: value 0.22u -> 100n
- C15: value 10u -> 100n
- C18: value 100n -> 1u
- C19: value 10u -> 1u
- C20: value 10n (25V) -> 10n
- C3: value 4.7u -> 100n
- C7: value 100n -> (none)
- C8: value 1u -> (none)
- renumbered U$1 to U1, U$12 to U2, U$13 to U3, U$4 to XTAL1, U$6 to RST, U$7 to BOOT
Connections:
- net N$8 renamed BOOT
- removed net DEN_GYRO: U3.DEN_G
- removed net DRDY_GYRO: U3.DRDY_G
- removed net I2C-1_SCL: U2.SCL
- removed net I2C-1_SDA: U2.SDA
- removed net INT1_ACCL: U3.INT1_A
- removed net INT1_GYRO: U3.INT1_G
- removed net INT2_ACCL: U3.INT2_A
- removed net LSM303-INT2: U2.INT2
- removed net N$7: C12.1, R1.1, RST.P$2, U1G$1.!RST
- removed net VDDA: C8.1, C9.1, U1G$1.VDDA
- new net !RST: C9.1, P2.!RST, R1.1, RST.P$2, U1G$1.!RST
- new net DM: P1.2, U1G$2.PORTA_11
- new net DP: P1.3, U1G$2.PORTA_12
- new net GPS_3DFIX: U1G$4.PORTC_11, U5.3D-FIX
- new net GPS_ENABLE: U1G$4.PORTC_10, U5.ENABLE
- new net GPS_RXD: R4.2, U1G$2.PORTA_2
- new net GPS_TXD: R3.2, U1G$2.PORTA_3
- new net I2C_SCL: R5.2, R8.1, U2.SCL, U4.SCL
- new net I2C_SDA: R6.2, R7.1, U2.SDA, U4.SDA
- new net LSM303_INT2: U1G$4.PORTC_2, U2.INT2
- new net LSM330_DEN_GYRO: U1G$4.PORTC_3, U3.DEN_G
- new net LSM330_DRDY_GYRO: U1G$4.PORTC_4, U3.DRDY_G
- new net LSM330_INT1_ACCL: U1G$4.PORTC_6, U3.INT1_A
- new net LSM330_INT1_GYRO: U1G$4.PORTC_5, U3.INT1_G
- new net LSM330_INT2_ACCL: U1G$4.PORTC_7, U3.INT2_A
- new net MPL311_P_INT1: U1G$4.PORTC_8, U4.INT1
- new net MPL311_P_INT2: U1G$4.PORTC_9, U4.INT2
- new net N$11: C16.1, U4.CAP
- new net N$14: R3.1, U5.TXD
- new net N$15: R4.1, U5.RXD
- new net N$18: C18.1, U5.VBACKUP
- new net PB8: R5.1, U1G$3.PORTB_8
- new net PB9: R6.1, U1G$3.PORTB_9
- new net SWCLK: P2.SWCLK, U1G$2.PORTA_14
- new net SWDIO: P2.SWDIO, U1G$2.PORTA_13
- new net VDD_5: C21.1, P1.1, P3.VDD_5P0V, U1G$2.PORTA_9, U6.IN
- new net VDD_GPS: C19.1, C20.1, L1.2, U5.VDD
- net GND: now also C14.2, C21.2, C22.2, P1.5, P1.S1, P2.GND, P3.GND, U4.VSS, U5.VSS, U6.GND; no longer C12.2
- net LSM303_DRDY: now also U1G$4.PORTC_0
- net LSM303_INT1: now also U1G$4.PORTC_1
- net N$10: now also C13.1; no longer C20.1
- net N$3: now also C12.1; no longer C14.1
- net N$4: now also C8.1; no longer C10.1
- net N$5: now also C12.2; no longer C14.2
- net N$6: now also C7.1; no longer C11.1
- net N$9: now also C10.1; no longer C13.1
- net SPI_CLK: now also U1G$2.PORTA_5
- net SPI_CS_ACCL: now also U1G$2.PORTA_0
- net SPI_CS_GYRO: now also U1G$2.PORTA_1
- net SPI_MISO: now also U1G$2.PORTA_6
- net SPI_MOSI: now also U1G$2.PORTA_7
- net VDD: now also C11.1, C14.1, C22.1, L1.1, P2.VDD_T, P3.VDD_3P3V, R7.2, R8.2, U1G$1.VDDA, U4.VDD, U4.VDD_IO, U6.OUT; no longer C16.1, C18.1, C19.1, C7.1
Other:
- note added: "Approx 110uA during operation"
- note added: "Approx 2mA during operation"
- note added: "Approx 50mA during operation"
- note added: "Approx 7mA during operation"
- note added: "I2C"
- note added: "USB"
- note removed: "100n cap should be close to VDDA pin."

Commit message: Changed all small caps, and all res to 0402. Large caps are 0805. Ripped all routing to start over again
Parts:
- C11, C12, C13, C14, C15, C16, C17, C20, C3, C4, C5, C6, C7, C8, C9: device resistor:C-EUC0805 -> resistor:C-EUC0402
- R1, R2, R3, R4, R5, R6, R7, R8: device resistor:R-EU_R0805 -> resistor:R-EU_R0402
Changed lines of the file:
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@@
 <part name="C1" library="resistor" deviceset="C-EU" device="C0805" value="2.2u"/>
 <part name="C2" library="resistor" deviceset="C-EU" device="C0805" value="2.2u"/>
-<part name="C3" library="resistor" deviceset="C-EU" device="C0805" value="100n"/>
-<part name="C4" library="resistor" deviceset="C-EU" device="C0805" value="100n"/>
-<part name="C5" library="resistor" deviceset="C-EU" device="C0805" value="100n"/>
-<part name="C6" library="resistor" deviceset="C-EU" device="C0805" value="100n"/>
+<part name="C3" library="resistor" deviceset="C-EU" device="C0402" value="100n"/>
+<part name="C4" library="resistor" deviceset="C-EU" device="C0402" value="100n"/>
+<part name="C5" library="resistor" deviceset="C-EU" device="C0402" value="100n"/>
+<part name="C6" library="resistor" deviceset="C-EU" device="C0402" value="100n"/>
 <part name="U$2" library="frames" deviceset="A4_L" device="">
 <attribute name="SHEET_NAME" value="stm32 Pwr/Rst"/>
@@
 </part>
 <part name="XTAL1" library="misc_devices" deviceset="XTAL_5X3P2" device=""/>
-<part name="C8" library="resistor" deviceset="C-EU" device="C0805"/>
-<part name="C7" library="resistor" deviceset="C-EU" device="C0805"/>
+<part name="C8" library="resistor" deviceset="C-EU" device="C0402"/>
+<part name="C7" library="resistor" deviceset="C-EU" device="C0402"/>
 <part name="U$5" library="frames" deviceset="A4_L" device="">
 <attribute name="SHEET_NAME" value="Interfaces"/>
@@
 <part name="RST" library="misc_devices" deviceset="OMRON_B3FS_1000" device=""/>
 <part name="BOOT" library="misc_devices" deviceset="OMRON_B3FS_1000" device=""/>
-<part name="R1" library="resistor" deviceset="R-EU_" device="R0805" value="10k"/>
-<part name="R2" library="resistor" deviceset="R-EU_" device="R0805" value="10k"/>
-<part name="C9" library="resistor" deviceset="C-EU" device="C0805" value="100n"/>
+<part name="R1" library="resistor" deviceset="R-EU_" device="R0402" value="10k"/>
+<part name="R2" library="resistor" deviceset="R-EU_" device="R0402" value="10k"/>
+<part name="C9" library="resistor" deviceset="C-EU" device="C0402" value="100n"/>
 <part name="U$8" library="frames" deviceset="A4_L" device="">
 <attribute name="SHEET_NAME" value="Accl / Mag"/>
@@
 <part name="U2" library="sensors" deviceset="LSM303DLHC" device=""/>
 <part name="C10" library="resistor" deviceset="C-EU" device="C0805" value="4.7u"/>
-<part name="C12" library="resistor" deviceset="C-EU" device="C0805" value="0.22u"/>
-<part name="C11" library="resistor" deviceset="C-EU" device="C0805" value="100n"/>
+<part name="C12" library="resistor" deviceset="C-EU" device="C0402" value="0.22u"/>
+<part name="C11" library="resistor" deviceset="C-EU" device="C0402" value="100n"/>
 <part name="U3" library="sensors" deviceset="LSM330DLC" device=""/>
-<part name="C15" library="resistor" deviceset="C-EU" device="C0805" value="100n"/>
-<part name="C14" library="resistor" deviceset="C-EU" device="C0805" value="100n"/>
-<part name="C13" library="resistor" deviceset="C-EU" device="C0805" value="10n (25V)"/>
+<part name="C15" library="resistor" deviceset="C-EU" device="C0402" value="100n"/>
+<part name="C14" library="resistor" deviceset="C-EU" device="C0402" value="100n"/>
+<part name="C13" library="resistor" deviceset="C-EU" device="C0402" value="10n (25V)"/>
 <part name="U4" library="sensors" deviceset="MPL3115A2" device=""/>
-<part name="C17" library="resistor" deviceset="C-EU" device="C0805" value="100n"/>
-<part name="C16" library="resistor" deviceset="C-EU" device="C0805" value="100n"/>
+<part name="C17" library="resistor" deviceset="C-EU" device="C0402" value="100n"/>
+<part name="C16" library="resistor" deviceset="C-EU" device="C0402" value="100n"/>
 <part name="U5" library="sensors" deviceset="MTK-3329" device=""/>
 <part name="L1" library="resistor" deviceset="R-EU_" device="R0603" value="MLB-160808-0060PQ"/>
-<part name="R3" library="resistor" deviceset="R-EU_" device="R0805" value="330R"/>
-<part name="R4" library="resistor" deviceset="R-EU_" device="R0805" value="330R"/>
+<part name="R3" library="resistor" deviceset="R-EU_" device="R0402" value="330R"/>
+<part name="R4" library="resistor" deviceset="R-EU_" device="R0402" value="330R"/>
 <part name="C19" library="resistor" deviceset="C-EU" device="C0805" value="1u"/>
 <part name="C18" library="resistor" deviceset="C-EU" device="C0805" value="1u"/>
-<part name="C20" library="resistor" deviceset="C-EU" device="C0805" value="10n"/>
+<part name="C20" library="resistor" deviceset="C-EU" device="C0402" value="10n"/>
 <part name="U$16" library="frames" deviceset="A4_L" device="">
 <attribute name="SHEET_NAME" value="Power"/>
@@
 <part name="C22" library="resistor" deviceset="C-EU" device="C0805" value="10u"/>
 <part name="P1" library="connectors" deviceset="USB_MICRO_AB" device=""/>
-<part name="R5" library="resistor" deviceset="R-EU_" device="R0805" value="100"/>
-<part name="R6" library="resistor" deviceset="R-EU_" device="R0805" value="100"/>
-<part name="R7" library="resistor" deviceset="R-EU_" device="R0805" value="4k7"/>
-<part name="R8" library="resistor" deviceset="R-EU_" device="R0805" value="4k7"/>
+<part name="R5" library="resistor" deviceset="R-EU_" device="R0402" value="100"/>
+<part name="R6" library="resistor" deviceset="R-EU_" device="R0402" value="100"/>
+<part name="R7" library="resistor" deviceset="R-EU_" device="R0402" value="4k7"/>
+<part name="R8" library="resistor" deviceset="R-EU_" device="R0402" value="4k7"/>
 <part name="P2" library="connectors" deviceset="ST_LINK" device=""/>
 <part name="P3" library="connectors" deviceset="PWR3" device=""/>

Commit message: Cleanup of power and layout
Parts:
- added P4: SPI_EXT, connectors:SPI_EXT
Connections:
- new net SPIEXT_CLK: P4.CLK, U1G$3.PORTB_13
- new net SPIEXT_MISO: P4.MISO, U1G$3.PORTB_14
- new net SPIEXT_MOSI: P4.MOSI, U1G$3.PORTB_15
- new net SPIEXT_NSS: P4.NSS, U1G$3.PORTB_12
- net GND: now also P4.GND
Changed lines of the file:
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@@
 <part name="P2" library="connectors" deviceset="ST_LINK" device=""/>
 <part name="P3" library="connectors" deviceset="PWR3" device=""/>
+<part name="P4" library="connectors" deviceset="SPI_EXT" device=""/>
 </parts>
 <sheets>
@@
 </segment>
 </net>
+<net name="SPIEXT_NSS" class="0">
+<segment>
+<pinref part="U1" gate="G$3" pin="PORTB_12"/>
+<wire x1="127" y1="127" x2="116.84" y2="127" width="0.1524" layer="91"/>
+<label x="111.76" y="127" size="1.778" layer="95"/>
+</segment>
+</net>
+<net name="SPIEXT_CLK" class="0">
+<segment>
+<pinref part="U1" gate="G$3" pin="PORTB_13"/>
+<wire x1="127" y1="132.08" x2="116.84" y2="132.08" width="0.1524" layer="91"/>
+<label x="111.76" y="132.08" size="1.778" layer="95"/>
+</segment>
+</net>
+<net name="SPIEXT_MISO" class="0">
+<segment>
+<pinref part="U1" gate="G$3" pin="PORTB_14"/>
+<wire x1="127" y1="137.16" x2="116.84" y2="137.16" width="0.1524" layer="91"/>
+<label x="111.76" y="137.16" size="1.778" layer="95"/>
+</segment>
+</net>
+<net name="SPIEXT_MOSI" class="0">
+<segment>
+<pinref part="U1" gate="G$3" pin="PORTB_15"/>
+<wire x1="127" y1="142.24" x2="116.84" y2="142.24" width="0.1524" layer="91"/>
+<label x="111.76" y="142.24" size="1.778" layer="95"/>
+</segment>
+</net>
 </nets>
 </sheet>
@@
 <instance part="P2" gate="G$1" x="55.88" y="38.1"/>
 <instance part="P3" gate="G$1" x="142.24" y="132.08"/>
+<instance part="P4" gate="G$1" x="142.24" y="78.74"/>
 </instances>
 <busses>
@@
 <label x="127" y="137.16" size="1.778" layer="95"/>
 </segment>
+<segment>
+<pinref part="P4" gate="G$1" pin="GND"/>
+<wire x1="139.7" y1="91.44" x2="129.54" y2="91.44" width="0.1524" layer="91"/>
+<label x="124.46" y="91.44" size="1.778" layer="95"/>
+</segment>
 </net>
 <net name="SWCLK" class="0">
@@
 </segment>
 </net>
+<net name="SPIEXT_CLK" class="0">
+<segment>
+<pinref part="P4" gate="G$1" pin="CLK"/>
+<wire x1="139.7" y1="81.28" x2="129.54" y2="81.28" width="0.1524" layer="91"/>
+<label x="124.46" y="81.28" size="1.778" layer="95"/>
+</segment>
+</net>
+<net name="SPIEXT_MOSI" class="0">
+<segment>
+<pinref part="P4" gate="G$1" pin="MOSI"/>
+<wire x1="139.7" y1="83.82" x2="129.54" y2="83.82" width="0.1524" layer="91"/>
+<label x="124.46" y="83.82" size="1.778" layer="95"/>
+</segment>
+</net>
+<net name="SPIEXT_MISO" class="0">
+<segment>
+<pinref part="P4" gate="G$1" pin="MISO"/>
+<wire x1="139.7" y1="86.36" x2="129.54" y2="86.36" width="0.1524" layer="91"/>
+<label x="124.46" y="86.36" size="1.778" layer="95"/>
+</segment>
+</net>
+<net name="SPIEXT_NSS" class="0">
+<segment>
+<pinref part="P4" gate="G$1" pin="NSS"/>
+<wire x1="139.7" y1="88.9" x2="129.54" y2="88.9" width="0.1524" layer="91"/>
+<label x="124.46" y="88.9" size="1.778" layer="95"/>
+</segment>
+</net>
