File: hw/projects/IMU_NoPilot/IMU_NoPilot.brd (EAGLE design)
At the start: 30 x 45 mm, 44 parts, among them P1 USB_MICRO_AB, P2 ST_LINK, P3 PWR3, P4 SPI_EXT, U1 STM32F4XX_64, U2 LSM303DLHC, U3 LSM330DLC, U4 MPL3115A2, U5 MTK-3329, U6 MCP1825

Commit message: Autoroute complete. Looks good
Parts:
- moved P3 0.50 mm to (27.9, 22.5)
Routing:
- net !RST: track 12.8 -> 64.5 mm, vias 1 -> 2
- net MPL311_P_INT2: track 0.00 -> 44.8 mm, vias 0 -> 2
- net LSM303_DRDY: track 0.00 -> 41.4 mm, vias 0 -> 2
- net GPS_TXD: track 0.00 -> 34.4 mm, vias 0 -> 1
- net I2C_SCL: track 0.00 -> 32.5 mm, vias 0 -> 2
- net SPI_CS_ACCL: track 0.00 -> 31.4 mm, vias 0 -> 2
- net MPL311_P_INT1: track 0.00 -> 30.2 mm, vias 0 -> 2
- net I2C_SDA: track 0.00 -> 23.4 mm, vias 0 -> 1
- net SPI_MOSI: track 0.00 -> 23.1 mm, vias 0 -> 2
- net LSM303_INT2: track 0.00 -> 22.0 mm, vias 0 -> 4
- net LSM330_DEN_GYRO: track 0.00 -> 20.4 mm, vias 0 -> 4
- net GPS_RXD: track 0.00 -> 19.6 mm, vias 0 -> 3
- net BOOT: track 9.95 -> 29.3 mm
- net LSM303_INT1: track 0.00 -> 19.3 mm, vias 0 -> 2
- net LSM330_INT1_ACCL: track 0.00 -> 19.2 mm, vias 0 -> 2
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- added copper zone on layer 1, net GND
- added copper zone on layer 16, net GND
Other:
- board text added: "http://www.lentic.net"
